Commit message: Fixed closed loop moment control in 03. Organized robot models in all controllers. Revised sensor and control point positions

File: 01-dual_proxy_motion_robot/panda_arm.urdf (robot description, URDF)
Before this commit: robot panda, 9 links, 8 joints
Joints:
- joint joint_fixed: origin xyz=0 0 0.13 rpy=0 0 0 -> xyz=0 0 0.142 rpy=0 0 0

File: 03-dual_proxy_surface_alignment_robot/panda_arm.urdf (robot description, URDF)
Before this commit: robot panda, 9 links, 8 joints
Links:
- link end_effector: geometry collision cylinder length=0.09 radius=0.04; visual cylinder length=0.09 radius=0.04
Joints:
- joint joint_fixed: origin xyz=0 0 0.105 rpy=0 0 0 -> xyz=0 0 0.107 rpy=0 0 0

File: 04-unified_motion_force/panda_arm.urdf (robot description, URDF)
Before this commit: robot panda, 9 links, 8 joints
Joints:
- joint joint_fixed: origin xyz=0 0 0.14 rpy=0 0 0 -> xyz=0 0 0.142 rpy=0 0 0
