Commit message: Revised control point. Fixed rotation matrix from sensor to link for tool calibration

File: 03-dual_proxy_surface_alignment_robot/panda_arm.urdf (robot description, URDF)
Before this commit: robot panda, 9 links, 8 joints
Links:
- link end_effector: geometry collision cylinder length=0.153 radius=0.04; visual cylinder length=0.153 radius=0.04
