Commit message: hand working for demo 03 as well

File: 03-dual_proxy_surface_alignment_robot/panda_arm_allegro.urdf (robot description, URDF)
Before this commit: robot panda, 8 links, 7 joints
Links:
- added link end_effector, mass 0.5; collision box size=0.1 0.1 0.1; visual box size=0.1 0.1 0.1
- added link link_0, mass 0.0119; collision mesh filename=../../../Model/allegro/link_0.0.obj; visual mesh filename=../../../Model/allegro/link_0.0.obj
- added link link_1, mass 0.065; collision mesh filename=../../../Model/allegro/link_1.0.obj; visual mesh filename=../../../Model/allegro/link_1.0.obj
- added link link_10, mass 0.0355; collision mesh filename=../../../Model/allegro/link_2.0.obj; visual mesh filename=../../../Model/allegro/link_2.0.obj
- added link link_11, mass 0.0096; collision mesh filename=../../../Model/allegro/link_3.0.obj; visual mesh filename=../../../Model/allegro/link_3.0.obj
- added link link_11_tip, mass 0.0168; collision sphere radius=0.012; visual mesh filename=../../../Model/allegro/link_3.0_tip.obj
- added link link_12, mass 0.0176; collision mesh filename=../../../Model/allegro/link_12.0_right.obj; visual mesh filename=../../../Model/allegro/link_12.0_right.obj
- added link link_13, mass 0.0119; collision mesh filename=../../../Model/allegro/link_13.0.obj; visual mesh filename=../../../Model/allegro/link_13.0.obj
- added link link_14, mass 0.038; collision mesh filename=../../../Model/allegro/link_14.0.obj; visual mesh filename=../../../Model/allegro/link_14.0.obj
- added link link_15, mass 0.0388; collision mesh filename=../../../Model/allegro/link_15.0.obj; visual mesh filename=../../../Model/allegro/link_15.0.obj
- added link link_15_tip, mass 0.0168; collision sphere radius=0.012; visual mesh filename=../../../Model/allegro/link_15.0_tip.obj
- added link link_2, mass 0.0355; collision mesh filename=../../../Model/allegro/link_2.0.obj; visual mesh filename=../../../Model/allegro/link_2.0.obj
- added link link_3, mass 0.0096; collision mesh filename=../../../Model/allegro/link_3.0.obj; visual mesh filename=../../../Model/allegro/link_3.0.obj
- added link link_3_tip, mass 0.0168; collision sphere radius=0.012; visual mesh filename=../../../Model/allegro/link_3.0_tip.obj
- added link link_4, mass 0.0119; collision mesh filename=../../../Model/allegro/link_0.0.obj; visual mesh filename=../../../Model/allegro/link_0.0.obj
- added link link_5, mass 0.065; collision mesh filename=../../../Model/allegro/link_1.0.obj; visual mesh filename=../../../Model/allegro/link_1.0.obj
- added link link_6, mass 0.0355; collision mesh filename=../../../Model/allegro/link_2.0.obj; visual mesh filename=../../../Model/allegro/link_2.0.obj
- added link link_7, mass 0.0096; collision mesh filename=../../../Model/allegro/link_3.0.obj; visual mesh filename=../../../Model/allegro/link_3.0.obj
- added link link_7_tip, mass 0.0168; collision sphere radius=0.012; visual mesh filename=../../../Model/allegro/link_3.0_tip.obj
- added link link_8, mass 0.0119; collision mesh filename=../../../Model/allegro/link_0.0.obj; visual mesh filename=../../../Model/allegro/link_0.0.obj
- added link link_9, mass 0.065; collision mesh filename=../../../Model/allegro/link_1.0.obj; visual mesh filename=../../../Model/allegro/link_1.0.obj
- added link palm_link, mass 0.4154; collision box size=0.0407 0.1125 0.093; visual mesh filename=../../../Model/allegro/base_link.obj
Joints:
- added joint hand_connection: type fixed, parent link7, child palm_link, origin xyz=0.05 0 0.135 rpy=3.1415926535 -1.57079632675 0
- added joint joint_0: type revolute, parent palm_link, child link_0, origin xyz=0 0.0435 -0.001542 rpy=-0.08726646255 0 0, axis 0 0 1, limit lower=-0.47 upper=0.47 effort=0.7 velocity=7
- added joint joint_1: type revolute, parent link_0, child link_1, origin xyz=0 0 0.0164, axis 0 1 0, limit lower=-0.196 upper=1.61 effort=0.7 velocity=7
- added joint joint_10: type revolute, parent link_9, child link_10, origin xyz=0 0 0.054, axis 0 1 0, limit lower=-0.174 upper=1.709 effort=0.7 velocity=7
- added joint joint_11: type revolute, parent link_10, child link_11, origin xyz=0 0 0.0384, axis 0 1 0, limit lower=-0.227 upper=1.618 effort=0.7 velocity=7
- added joint joint_11_tip: type fixed, parent link_11, child link_11_tip, origin xyz=0 0 0.0267 rpy=0 0 0
- added joint joint_12: type revolute, parent palm_link, child link_12, origin xyz=-0.0182 0.019333 -0.045987 rpy=0 -1.65806278845 -1.5707963259, axis 1 0 0, limit lower=0.263 upper=1.396 effort=0.7 velocity=7
- added joint joint_13: type revolute, parent link_12, child link_13, origin xyz=-0.027 0.005 0.0399, axis 0 0 1, limit lower=-0.105 upper=1.163 effort=0.7 velocity=7
- added joint joint_14: type revolute, parent link_13, child link_14, origin xyz=0 0 0.0177, axis 0 1 0, limit lower=-0.189 upper=1.644 effort=0.7 velocity=7
- added joint joint_15: type revolute, parent link_14, child link_15, origin xyz=0 0 0.0514, axis 0 1 0, limit lower=-0.162 upper=1.719 effort=0.7 velocity=7
- added joint joint_15_tip: type fixed, parent link_15, child link_15_tip, origin xyz=0 0 0.0423 rpy=0 0 0
- added joint joint_2: type revolute, parent link_1, child link_2, origin xyz=0 0 0.054, axis 0 1 0, limit lower=-0.174 upper=1.709 effort=0.7 velocity=7
- added joint joint_3: type revolute, parent link_2, child link_3, origin xyz=0 0 0.0384, axis 0 1 0, limit lower=-0.227 upper=1.618 effort=0.7 velocity=7
- added joint joint_3_tip: type fixed, parent link_3, child link_3_tip, origin xyz=0 0 0.0267 rpy=0 0 0
- added joint joint_4: type revolute, parent palm_link, child link_4, origin xyz=0 0 0.0007 rpy=0.0 0 0, axis 0 0 1, limit lower=-0.47 upper=0.47 effort=0.7 velocity=7
- added joint joint_5: type revolute, parent link_4, child link_5, origin xyz=0 0 0.0164, axis 0 1 0, limit lower=-0.196 upper=1.61 effort=0.7 velocity=7
- added joint joint_6: type revolute, parent link_5, child link_6, origin xyz=0 0 0.054, axis 0 1 0, limit lower=-0.174 upper=1.709 effort=0.7 velocity=7
- added joint joint_7: type revolute, parent link_6, child link_7, origin xyz=0 0 0.0384, axis 0 1 0, limit lower=-0.227 upper=1.618 effort=0.7 velocity=7
- added joint joint_7_tip: type fixed, parent link_7, child link_7_tip, origin xyz=0 0 0.0267 rpy=0 0 0
- added joint joint_8: type revolute, parent palm_link, child link_8, origin xyz=0 -0.0435 -0.001542 rpy=0.08726646255 0 0, axis 0 0 1, limit lower=-0.47 upper=0.47 effort=0.7 velocity=7
- added joint joint_9: type revolute, parent link_8, child link_9, origin xyz=0 0 0.0164, axis 0 1 0, limit lower=-0.196 upper=1.61 effort=0.7 velocity=7
- added joint joint_fixed: type fixed, parent link7, child end_effector, origin xyz=0 0 0.157 rpy=0 0 0
