Commit message: Added adjustable EE frame to surface alignment example

File: xx-unified_motion_force/panda_arm.urdf (robot description, URDF)
Before this commit: robot panda, 9 links, 8 joints
Links:
- link end_effector: geometry collision sphere radius=0.035; visual sphere radius=0.035
Joints:
- joint joint_fixed: origin xyz=0 0 0.157 rpy=0 0 0 -> xyz=0 0 0.142 rpy=0 0 0
