Commit message: Integrated optitrack pose following in lead controller

File: lead_control/panda_arm.urdf (robot description, URDF)
Before this commit: robot panda, 9 links, 8 joints
Joints:
- joint joint_fixed: origin xyz=0 0 0.142 rpy=0 0 0 -> xyz=0 0 0.107 rpy=0 0 0

File: lead_control/panda_arm_allegro.urdf (robot description, URDF)
Before this commit: robot panda, 30 links, 29 joints
Links:
- link link_12: geometry collision mesh filename=../../../Model/allegro/link_12.0_right.obj; visual mesh filename=../../../Model/allegro/link_12.0_right.obj
- link palm_link: geometry collision box size=0.0407 0.1125 0.093; visual mesh filename=../../../Model/allegro/base_link.obj
Joints:
- joint joint_12: origin xyz=-0.0182 -0.019333 -0.045987 rpy=0 -1.65806278845 1.5707963259 -> xyz=-0.0182 0.019333 -0.045987 rpy=0 -1.65806278845 -1.5707963259
- joint joint_13: origin xyz=-0.027 -0.005 0.0399 -> xyz=-0.027 0.005 0.0399
- joint joint_fixed: origin xyz=0 0 0.142 rpy=0 0 0 -> xyz=0 0 0.107 rpy=0 0 0

File: lead_control/panda_arm_allegro_left.urdf (robot description, URDF)
Before this commit: robot panda, 30 links, 29 joints
Links:
- link link_12: geometry collision mesh filename=../../../Model/allegro/link_12.0_left.obj; visual mesh filename=../../../Model/allegro/link_12.0_left.obj
- link palm_link: geometry collision box size=0.0407 0.1125 0.093; visual mesh filename=../../../Model/allegro/base_link_left.obj
Joints:
- joint joint_12: origin xyz=-0.0182 0.019333 -0.045987 rpy=0 -1.65806278845 -1.5707963259 -> xyz=-0.0182 -0.019333 -0.045987 rpy=0 -1.65806278845 1.5707963259
- joint joint_13: origin xyz=-0.027 0.005 0.0399 -> xyz=-0.027 -0.005 0.0399
- joint joint_fixed: origin xyz=0 0 0.142 rpy=0 0 0 -> xyz=0 0 0.107 rpy=0 0 0
